File: test_board/test_board.kicad_sch (KiCad schematic)
At the start: 8 parts, among them IC1 TC118S, J1 MotorConnection, U1 ACS712xLCTR-05B

Commit message: Improved MG-X
Parts:
- added J3: PowerSupply, TerminalBlock:TerminalBlock_bornier-2_P5.08mm, symbol Connector_Generic:Conn_01x02
Connections:
- net GND: now also J3.2 (Pin_2)
- net VCC: now also J3.1 (Pin_1)
Other:
- moved on the sheet: C4
Changed lines of the file:
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@@
+	)
+	(junction
+		(at 88.9 109.22)
+		(diameter 0)
+		(color 0 0 0 0)
 	)
 	(junction
@@
 	)
 	(junction
-		(at 88.9 111.76)
-		(diameter 0)
-		(color 0 0 0 0)
-	)
-	(junction
 		(at 154.94 105.41)
 		(diameter 0)
@@
 	)
 	(junction
+		(at 106.68 71.12)
+		(diameter 0)
+		(color 0 0 0 0)
+	)
+	(junction
 		(at 154.94 85.09)
 		(diameter 0)
@@
 	(wire
 		(pts
-			(xy 88.9 104.14) (xy 88.9 111.76)
+			(xy 88.9 104.14) (xy 88.9 109.22)
 		)
 		(stroke
@@
 	(wire
 		(pts
-			(xy 106.68 88.9) (xy 106.68 68.58)
-		)
-		(stroke
-			(width 0)
-			(type default)
-		)
-	)
-	(wire
-		(pts
-			(xy 74.93 96.52) (xy 74.93 100.33)
+			(xy 113.03 73.66) (xy 113.03 76.2)
+		)
+		(stroke
+			(width 0)
+			(type default)
+		)
+	)
+	(wire
+		(pts
+			(xy 106.68 88.9) (xy 106.68 71.12)
+		)
+		(stroke
+			(width 0)
+			(type default)
+		)
+	)
+	(wire
+		(pts
+			(xy 74.93 96.52) (xy 74.93 99.06)
 		)
 		(stroke
@@
 	(wire
 		(pts
+			(xy 88.9 109.22) (xy 88.9 113.03)
+		)
+		(stroke
+			(width 0)
+			(type default)
+		)
+	)
+	(wire
+		(pts
 			(xy 143.51 96.52) (xy 143.51 111.76)
 		)
@@
 	(wire
 		(pts
+			(xy 106.68 71.12) (xy 106.68 68.58)
+		)
+		(stroke
+			(width 0)
+			(type default)
+		)
+	)
+	(wire
+		(pts
 			(xy 138.43 85.09) (xy 138.43 91.44)
 		)
@@
 	(wire
 		(pts
-			(xy 88.9 111.76) (xy 88.9 113.03)
-		)
-		(stroke
-			(width 0)
-			(type default)
-		)
-	)
-	(wire
-		(pts
 			(xy 99.06 99.06) (xy 110.49 99.06)
 		)
@@
 	(wire
 		(pts
+			(xy 106.68 71.12) (xy 115.57 71.12)
+		)
+		(stroke
+			(width 0)
+			(type default)
+		)
+	)
+	(wire
+		(pts
 			(xy 167.64 96.52) (xy 167.64 105.41)
 		)
@@
 	(wire
 		(pts
-			(xy 74.93 111.76) (xy 88.9 111.76)
+			(xy 74.93 109.22) (xy 88.9 109.22)
 		)
 		(stroke
@@
 	(wire
 		(pts
-			(xy 74.93 107.95) (xy 74.93 111.76)
+			(xy 74.93 106.68) (xy 74.93 109.22)
 		)
 		(stroke
@@
 		(pts
 			(xy 99.06 88.9) (xy 106.68 88.9)
+		)
+		(stroke
+			(width 0)
+			(type default)
+		)
+	)
+	(wire
+		(pts
+			(xy 115.57 73.66) (xy 113.03 73.66)
 		)
 		(stroke
@@
 				(path "/4177eac5-413f-4b05-b79c-aa28993c8fbf"
 					(reference "#PWR01")
+					(unit 1)
+				)
+			)
+		)
+	)
+	(symbol
+		(lib_id "power:GND")
+		(at 113.03 76.2 0)
+		(unit 1)
+		(exclude_from_sim no)
+		(in_bom yes)
+		(on_board yes)
+		(dnp no)
+		(fields_autoplaced yes)
+		(property "Reference" "#PWR08"
+			(at 113.03 82.55 0)
+			(effects
+				(font
+					(size 1.27 1.27)
+				)
+				(hide yes)
+			)
+		)
+		(property "Value" "GND"
+			(at 113.03 81.28 0)
+			(effects
+				(font
+					(size 1.27 1.27)
+				)
+			)
+		)
+		(property "Footprint" ""
+			(at 113.03 76.2 0)
+			(effects
+				(font
+					(size 1.27 1.27)
+				)
+				(hide yes)
+			)
+		)
+		(property "Datasheet" ""
+			(at 113.03 76.2 0)
+			(effects
+				(font
+					(size 1.27 1.27)
+				)
+				(hide yes)
+			)
+		)
+		(property "Description" "Power symbol creates a global label with name \"GND\" , ground"
+			(at 113.03 76.2 0)
+			(effects
+				(font
+					(size 1.27 1.27)
+				)
+				(hide yes)
+			)
+		)
+		(pin "1"
+		)
+		(instances
+			(project "test_board"
+				(path "/4177eac5-413f-4b05-b79c-aa28993c8fbf"
+					(reference "#PWR08")
+					(unit 1)
+				)
+			)
+		)
+	)
+	(symbol
+		(lib_id "Connector_Generic:Conn_01x02")
+		(at 120.65 71.12 0)
+		(unit 1)
+		(exclude_from_sim no)
+		(in_bom yes)
+		(on_board yes)
+		(dnp no)
+		(fields_autoplaced yes)
+		(property "Reference" "J3"
+			(at 123.19 71.1199 0)
+			(effects
+				(font
+					(size 1.27 1.27)
+				)
+				(justify left)
+				(hide yes)
+			)
+		)
+		(property "Value" "PowerSupply"
+			(at 123.19 73.6599 0)
+			(effects
+				(font
+					(size 1.27 1.27)
+				)
+				(justify left)
+				(hide yes)
+			)
+		)
+		(property "Footprint" "TerminalBlock:TerminalBlock_bornier-2_P5.08mm"
+			(at 120.65 71.12 0)
+			(effects
+				(font
+					(size 1.27 1.27)
+				)
+				(hide yes)
+			)
+		)
+		(property "Datasheet" "~"
+			(at 120.65 71.12 0)
+			(effects
+				(font
+					(size 1.27 1.27)
+				)
+				(hide yes)
+			)
+		)
+		(property "Description" "Generic connector, single row, 01x02, script generated (kicad-library-utils/schlib/autogen/connector/)"
+			(at 120.65 71.12 0)
+			(effects
+				(font
+					(size 1.27 1.27)
+				)
+				(hide yes)
+			)
+		)
+		(pin "2"
+		)
+		(pin "1"
+		)
+		(instances
+			(project "test_board"
+				(path "/4177eac5-413f-4b05-b79c-aa28993c8fbf"
+					(reference "J3")
 					(unit 1)
 				)
@@
 	(symbol
 		(lib_id "Device:C")
-		(at 74.93 104.14 0)
+		(at 74.93 102.87 0)
 		(mirror y)
 		(unit 1)
@@
 		(dnp no)
 		(property "Reference" "C4"
-			(at 71.12 102.8699 0)
+			(at 71.12 101.5999 0)
 			(effects
 				(font
@@
 		)
 		(property "Value" "100nF"
-			(at 71.12 105.4099 0)
+			(at 71.12 104.1399 0)
 			(effects
 				(font
@@
 		)
 		(property "Footprint" "Capacitor_THT:C_Disc_D3.0mm_W2.0mm_P2.50mm"
-			(at 73.9648 107.95 0)
+			(at 73.9648 106.68 0)
 			(effects
 				(font
@@
 		)
 		(property "Datasheet" "~"
-			(at 74.93 104.14 0)
+			(at 74.93 102.87 0)
 			(effects
 				(font
@@
 		)
 		(property "Description" "Unpolarized capacitor"
-			(at 74.93 104.14 0)
+			(at 74.93 102.87 0)
 			(effects
 				(font
@@
 		(on_board yes)
 		(dnp no)
-		(fields_autoplaced yes)
 		(property "Reference" "C2"
 			(at 151.13 100.3299 0)
