File: match_x/match_x.kicad_pcb (KiCad board)
At the start: 2 copper layers, 17 x 20 mm, 17 parts, among them IC1 TC118S, J1 Conn_01x02, J2 Conn_01x03, J3 Conn_01x03, J4 Conn_01x06, U1 ATtiny88-A, U2 LD3985G18R_TSOT23, U3 MPU-6050, U4 ACS712xLCTR-05B

Commit message: Potenciometer installed
Parts:
- added U5: ATtiny861A-X, Package_SO:TSSOP-20_4.4x6.5mm_P0.65mm, F.Cu at (150.2, 101.6)
- IC1: footprint TC118S:SOIC127P600X155-8N -> Package_SO:SOIC-8_3.9x4.9mm_P1.27mm
- U1: value ATtiny88-A -> X9C104P; footprint Package_QFP:TQFP-32_7x7mm_P0.8mm -> Package_SO:SOIC-8_3.9x4.9mm_P1.27mm; moved to B.Cu
- moved U1 21.5 mm to (147.0, 80.5), turned to 180 degrees
- moved C2 7.06 mm to (139.0, 87.0)
- moved U4 4.24 mm to (152.0, 74.4), turned to 180 degrees
- moved C8 3.48 mm to (154.7, 96.2), turned to 180 degrees
- moved IC1 1.62 mm to (153.9, 81.0), turned to -90 degrees
- moved C5 0.97 mm to (158.3, 81.0)
- moved C7 0.39 mm to (152.8, 90.9)
- moved U3 0.39 mm to (156.5, 93.0)
- moved C4 0.37 mm to (145.8, 93.1)
- moved C6 0.37 mm to (144.7, 93.1)
- moved U2 0.37 mm to (148.3, 92.5)
- moved C3 0.37 mm to (150.8, 91.3)
- moved J2 0.31 mm to (158.5, 98.5)
Connections:
- U1 pad 4: +3.3V -> unconnected-(U1-VSS-Pad4)
- U1 pad 5: GND -> unconnected-(U1-VW/RW-Pad5)
