File: match_x/match_x.kicad_sch (KiCad schematic)
At the start: 17 parts, among them IC1 TC118S, J1 Conn_01x02, J2 Conn_01x03, J3 Conn_01x03, J4 Conn_01x06, U1 ATtiny88-A, U2 LD3985G18R_TSOT23, U3 MPU-6050, U4 ACS712xLCTR-05B

Commit message: Potenciometer installed
Parts:
- removed U1: ATtiny88-A, Package_QFP:TQFP-32_7x7mm_P0.8mm, symbol MCU_Microchip_ATtiny:ATtiny88-A
- added U1: X9C104P, Package_SO:SOIC-8_3.9x4.9mm_P1.27mm, symbol X9C104P:X9C104P
- added U5: ATtiny861A-X, Package_SO:TSSOP-20_4.4x6.5mm_P0.65mm, symbol MCU_Microchip_ATtiny:ATtiny861A-X
- U5: renamed from IC1; footprint SOIC127P600X155-8N -> Package_SO:SOIC-8_3.9x4.9mm_P1.27mm
Connections:
- net +3.3V: now also U5.5 (VCC)
- net ASEN: now also U5.7 (XTAL1/PB4)
- net BSEN: now also U5.9 (PB6)
- net CS: now also U5.14 (PA4)
- net CSEN: now also U5.8 (XTAL2/PB5)
- net GND: now also U5.6 (GND)
- net INA: now also U5.3 (PB2)
- net INB: now also U5.4 (PB3)
- net MISO: now also U5.18 (PA2)
- net MOSI: now also U5.19 (PA1)
- net SCK: now also U5.17 (AREF/PA3)
- net SCL: now also U5.1 (PB0)
- net SDA: now also U5.2 (PB1)
- no-connect marks 2 -> 1
Other:
- moved on the sheet: C7, C8, J2, J3, J4, U3
