File: sg_x/sg_x.kicad_pcb (KiCad board)
At the start: 2 copper layers, 9.8 x 13 mm, 7 parts, among them IC1 TC118S, J1 Conn_01x03, J2 Conn_01x04, U1 ATtiny25-20SS

Commit message: Minor changes
Parts:
- removed C5: 104pF, Capacitor_SMD:C_1206_3216Metric
- C2: value 100nF -> 4.7uF
- C3: value 104pF -> 100nF
- moved C3 2.32 mm to (162.1, 92.4), turned to 0 degrees
Routing:
- net Net-(IC1-OUTA): track 12.9 -> 6.52 mm
- net Net-(IC1-OUTB): track 20.6 -> 15.4 mm
- net VCC: track 15.0 -> 17.3 mm
Other:
- board size 9.8 x 13 mm -> 8.9 x 13 mm

Commit message: Commit the SG-X improved
Parts:
- C2: value 4.7uF -> 100nF; footprint Capacitor_SMD:C_1210_3225Metric -> Capacitor_SMD:C_0603_1608Metric
- C3: footprint Capacitor_SMD:C_1206_3216Metric -> Capacitor_SMD:C_0603_1608Metric
- moved C2 1.37 mm to (163.1, 100.4)
- moved C3 0.60 mm to (162.1, 91.8)
Routing:
- net VCC: track 17.3 -> 0.00 mm
- net Net-(IC1-OUTB): track 15.4 -> 0.00 mm
- net ADC0: track 10.1 -> 0.00 mm
- net /SCL: track 9.69 -> 0.00 mm, vias 1 -> 0
- net /INB: track 8.08 -> 0.00 mm, vias 1 -> 0
- net /SDA: track 6.95 -> 0.00 mm, vias 1 -> 0
- net Net-(IC1-OUTA): track 6.52 -> 0.00 mm
- net /INA: track 5.07 -> 0.00 mm, vias 1 -> 0
Other:
- board text added: "ADC"

Commit message: Minor changes
Parts:
- added J3: Conn_01x03, Connector_Servo_Driver:Connector_Servo_Driver_ADC, F.Cu at (162.1, 89.4)
- added U2: ACS712xLCTR-05B, Package_SO:SOIC-8_3.9x4.9mm_P1.27mm, B.Cu at (162.1, 93.2)
- IC1: footprint TC118S:SOIC127P600X155-8N -> Package_SO:SOIC-8_3.9x4.9mm_P1.27mm
- J1: value Conn_01x03 -> Conn_01x02
- J2: footprint Connector_Servo_Driver:Connector_Servo_Driver -> Connector_Servo_Driver:Connector_Servo_Driver_SMD; moved to F.Cu
- U1: value ATtiny25-20SS -> ATtiny84A-M; footprint Package_SO:SOIC-8_3.9x4.9mm_P1.27mm -> Package_DFN_QFN:QFN-20-1EP_4x4mm_P0.5mm_EP2.6x2.6mm
- moved C2 24.4 mm to (138.8, 97.9)
- moved U1 23.1 mm to (139.1, 94.5)
- moved IC1 2.21 mm to (162.1, 98.8)
- moved C3 2.14 mm to (162.1, 89.7), turned to 180 degrees
- moved J2 1.49 mm to (162.1, 100.4), turned to 0 degrees
- moved J1 0.34 mm to (162.1, 89.7)
Connections:
- IC1 pad 4: VCC -> Net-(IC1-VDD)
- J1 pad 1: Net-(IC1-OUTB) -> Net-(IC1-OUTA)
- J1 pad 2: ADC0 -> Net-(IC1-OUTB)
- U1 pad 2: /INB -> unconnected-(U1-PA3-Pad2)
- U1 pad 3: ADC0 -> unconnected-(U1-PA2-Pad3)
- U1 pad 4: GND -> unconnected-(U1-PA1-Pad4)
- U1 pad 5: /SDA -> unconnected-(U1-AREF/PA0-Pad5)
- U1 pad 6: /INA -> unconnected-(U1-NC-Pad6)
- U1 pad 7: /SCL -> unconnected-(U1-NC-Pad7)
- U1 pad 8: VCC -> GND
Routing:
- removed copper zone on B.Cu, net GND
- removed copper zone on F.Cu, net GND
Other:
- board size 8.9 x 13 mm -> 9 x 13 mm
- board text removed: "ADC"
- board text removed: "ATTiny85"
- board text removed: "GND"
- board text removed: "SCL"
- board text removed: "SDA"
- board text removed: "TC118S"
- board text removed: "VCC"
