File: sg_x/sg_x.kicad_sch (KiCad schematic)
At the start: 7 parts, among them IC1 TC118S, J1 Conn_01x03, J2 Conn_01x04, U1 ATtiny25-20SS

Commit message: Commit the SG-X improved
Parts:
- removed C5: 104pF, Capacitor_SMD:C_1206_3216Metric, symbol Device:C
- C2: footprint Capacitor_SMD:C_1210_3225Metric -> Capacitor_SMD:C_0603_1608Metric
- C3: value 104pF -> 100nF; footprint Capacitor_SMD:C_1206_3216Metric -> Capacitor_SMD:C_0603_1608Metric
Changed lines of the file:
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@@
-	)
-	(junction
-		(at 170.18 116.84)
-		(diameter 0)
-		(color 0 0 0 0)
 	)
 	(junction
@@
 	)
 	(junction
-		(at 170.18 96.52)
-		(diameter 0)
-		(color 0 0 0 0)
-	)
-	(junction
 		(at 153.67 96.52)
 		(diameter 0)
@@
 	)
 	(no_connect
-		(at 72.39 106.68)
+		(at 68.58 106.68)
 	)
 	(bus_entry
@@
 	(wire
 		(pts
-			(xy 185.42 102.87) (xy 185.42 96.52)
-		)
-		(stroke
-			(width 0)
-			(type default)
-		)
-	)
-	(wire
-		(pts
 			(xy 63.5 96.52) (xy 69.85 96.52)
 		)
@@
 	(wire
 		(pts
-			(xy 170.18 116.84) (xy 185.42 116.84)
-		)
-		(stroke
-			(width 0)
-			(type default)
-		)
-	)
-	(wire
-		(pts
 			(xy 204.47 54.61) (xy 204.47 59.69)
 		)
@@
 	(wire
 		(pts
-			(xy 170.18 96.52) (xy 185.42 96.52)
-		)
-		(stroke
-			(width 0)
-			(type default)
-		)
-	)
-	(wire
-		(pts
 			(xy 209.55 49.53) (xy 217.17 49.53)
 		)
@@
 	(wire
 		(pts
-			(xy 185.42 110.49) (xy 185.42 116.84)
-		)
-		(stroke
-			(width 0)
-			(type default)
-		)
-	)
-	(wire
-		(pts
-			(xy 72.39 106.68) (xy 63.5 106.68)
+			(xy 68.58 106.68) (xy 63.5 106.68)
 		)
 		(stroke
@@
 			)
 		)
-		(property "Value" "104pF"
+		(property "Value" "100nF"
 			(at 149.86 107.9499 0)
 			(effects
@@
 			)
 		)
-		(property "Footprint" "Capacitor_SMD:C_1206_3216Metric"
+		(property "Footprint" "Capacitor_SMD:C_0603_1608Metric"
 			(at 152.7048 110.49 0)
 			(effects
@@
 	)
 	(symbol
-		(lib_id "Device:C")
-		(at 185.42 106.68 0)
-		(unit 1)
-		(exclude_from_sim no)
-		(in_bom yes)
-		(on_board yes)
-		(dnp no)
-		(property "Reference" "C5"
-			(at 189.23 105.4099 0)
-			(effects
-				(font
-					(size 1.27 1.27)
-				)
-				(justify left)
-			)
-		)
-		(property "Value" "104pF"
-			(at 189.23 107.9499 0)
-			(effects
-				(font
-					(size 1.27 1.27)
-				)
-				(justify left)
-			)
-		)
-		(property "Footprint" "Capacitor_SMD:C_1206_3216Metric"
-			(at 186.3852 110.49 0)
-			(effects
-				(font
-					(size 1.27 1.27)
-				)
-				(hide yes)
-			)
-		)
-		(property "Datasheet" "~"
-			(at 185.42 106.68 0)
-			(effects
-				(font
-					(size 1.27 1.27)
-				)
-				(hide yes)
-			)
-		)
-		(property "Description" "Unpolarized capacitor"
-			(at 185.42 106.68 0)
-			(effects
-				(font
-					(size 1.27 1.27)
-				)
-				(hide yes)
-			)
-		)
-		(pin "2"
-		)
-		(pin "1"
-		)
-		(instances
-			(project "sg_x"
-				(path "/e6ca21f7-2fbf-4ce0-9422-134e489615d1"
-					(reference "C5")
-					(unit 1)
-				)
-			)
-		)
-	)
-	(symbol
 		(lib_id "power:VCC")
 		(at 48.26 81.28 0)
@@
 			)
 		)
-		(property "Footprint" "Capacitor_SMD:C_1210_3225Metric"
+		(property "Footprint" "Capacitor_SMD:C_0603_1608Metric"
 			(at 203.5048 54.61 0)
 			(effects

Commit message: Minor changes
Parts:
- removed J1: Conn_01x03, Connector_Servo_Driver:Connector_DC_Motor, symbol Connector_Generic:Conn_01x03
- removed U1: ATtiny25-20SS, Package_SO:SOIC-8_3.9x4.9mm_P1.27mm, symbol MCU_Microchip_ATtiny:ATtiny25-20SS
- added J1: Conn_01x02, Connector_Servo_Driver:Connector_DC_Motor, symbol Connector_Generic:Conn_01x02
- added J3: Conn_01x03, Connector_Servo_Driver:Connector_Servo_Driver_ADC, symbol Connector_Generic:Conn_01x03
- added U1: ATtiny84A-M, Package_DFN_QFN:QFN-20-1EP_4x4mm_P0.5mm_EP2.6x2.6mm, symbol MCU_Microchip_ATtiny:ATtiny84A-M
- added U2: ACS712xLCTR-05B, Package_SO:SOIC-8_3.9x4.9mm_P1.27mm, symbol Sensor_Current:ACS712xLCTR-05B
- IC1: footprint SOIC127P600X155-8N -> Package_SO:SOIC-8_3.9x4.9mm_P1.27mm
- J2: footprint Connector_Servo_Driver:Connector_Servo_Driver -> Connector_Servo_Driver:Connector_Servo_Driver_SMD
Connections:
- net GND: now also U1.21 (GND), U1.8 (GND), U2.5 (GND)
- net VCC: now also U1.9 (VCC), U2.1 (IP+), U2.2 (IP+), U2.8 (VCC); no longer IC1.4 (VDD)
- net at C3.1, IC1.8 (OUTA): now also J1.1 (Pin_1)
- net at C3.2, IC1.5 (OUTB): now also J1.2 (Pin_2)
- new net: IC1.4 (VDD), U2.3 (IP-), U2.4 (IP-)
- no-connect marks 1 -> 0
Other:
- moved on the sheet: C3, IC1
